Commit message: 2024 track implemented in simulator
Co-authored-by: Copilot <copilot@github.com>

File: model/robot.xacro (robot description, xacro)
@@ -5,10 +5,10 @@
 <!--Body Dimensions-->
 <xacro:property name="pi_const" value="3.14159265"/>
-<xacro:property name="a" value="1.0"/>
-<xacro:property name="b" value="0.3"/>
-<xacro:property name="c" value="0.6"/>
+<xacro:property name="a" value="0.25"/>
+<xacro:property name="b" value="0.2"/>
+<xacro:property name="c" value="0.2"/>
 <!--Wheel and Caster-->
-<xacro:property name="r" value="0.15"/>
-<xacro:property name="d" value="0.1"/>
+<xacro:property name="r" value="0.05"/>
+<xacro:property name="d" value="0.02"/>
 <xacro:property name="s1" value="${b/2+r}"/>
 <xacro:property name="s2" value="${2*r}"/>
